File: Documents/Wattmeter_V4/WattMeter_v4.brd (EAGLE design)
At the start: 58 x 27 mm, 77 parts, among them Q1 QUARTZ_3.58M_2PIN, U1 ADE7953, U10 PS2505, U11 SN74LVC1G3157DBVR, U2 PAM2305, U3 ISO7241, U4 SN74LVC, U5 PS2505, U6 PS2505, U7 SN74LVC, U8 SN6501, U9 TRANSFO_3.3

Commit message: Updated V4 board
Parts:
- removed U$1: BUFFER-NL17SZ125, arducoder:TSOP-5
- added R12, R29: 55k, SparkFun:0603-RES
- added R25, R32: 100k, SparkFun:0603-RES
- added R28, R7: 4.7k, SparkFun:0603-RES
- added R33: 4.7k, Nizanlib:0402-RES
- added U12: PS2505, wattmeter:PS2505
- R30, R31: value 255k -> 100k; device Nizanlib:0402-RES -> SparkFun:0603-RES
- U10, U6: device Damien_divers:4-SMD -> wattmeter:PS2505
- U5: value PS2505 -> NL17SZ125; device Damien_divers:4-SMD -> wattmeter:NL17SZ125
- moved R31 86.2 mm to (49.0, 28.4), turned to 180 degrees
- moved R30 85.9 mm to (49.0, 31.0), turned to 180 degrees
- moved U11 71.8 mm to (32.7, 27.5), turned to 90 degrees
- moved R27 65.9 mm to (25.1, 28.9), turned to 270 degrees
- moved U10 59.1 mm to (23.2, 28.6), turned to 180 degrees
- moved R26 56.3 mm to (6.50, 26.3), turned to 270 degrees
- moved J1 22.5 mm to (4.34, 7.98), turned to 90 degrees
- moved U6 10.0 mm to (23.1, 34.0)
- moved U5 7.38 mm to (9.75, 12.1), turned to 180 degrees
- moved JP3 7.21 mm to (59.4, 9.08)
- moved JP2 7.21 mm to (59.3, 20.6)
- moved JP4 7.21 mm to (59.4, 14.8)
- moved Q1 6.75 mm to (38.7, 20.5)
- moved C9 6.39 mm to (36.2, 7.02)
- moved C1 6.39 mm to (37.4, 17.4)
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Connections:
- removed net N$29: R10.1, U6.1
- new net AGND: C10.2, C11.1, C12.2, C13.1, C14.1, C17.2, C28.1, C29.2, C30.1, C31.2, C5.1, C6.2, C7.2, C8.2, R11.2, R17.1, R18.2, R19.2, R20.2, R9.1, U1.16
- new net CF1: U1.23
- new net CF2: U1.24
- new net N$35: R25.1, R30.2
- new net N$36: R12.1, R25.2
- new net N$37: R28.1, R29.2, U11.1
- new net N$38: R12.2, R7.2, U11.3
- new net N$39: R10.1, U10.1
- new net REVP: U1.20
- new net ZX: U1.1
- new net ZX_I: U1.21
- net CS: now also J1.1, U5.1; no longer J1.2, U$1.1
- net GND: now also J1.8, R33.1, U12.4, U5.3; no longer J1.9, U$1.3, U5.2
- net GNDI: now also R28.2, R7.1, U10.2, U12.1, U6.1; no longer C10.2, C11.1, C12.2, C13.1, C14.1, C17.2, C28.1, C29.2, C30.1, C31.2, C5.1, C6.2, C7.2, C8.2, R11.2, R17.1, R18.2, R19.2, R20.2, R9.1, U1.16, U10.1, U5.3, U6.2
- net IRQ: now also U10.4; no longer U6.4
- net MISO: now also U5.2; no longer U$1.2
- net MISO_OUT: now also J1.2; no longer J1.3, U$1.4
- net MOSI: now also J1.4; no longer J1.5
- net N$13: now also R31.2, R32.1; no longer R30.2, U11.3
- net N$22: now also R29.1, R32.2; no longer R31.2, U11.1
- net N$25: now also U12.3; no longer U5.1
- net RESET: now also J1.6; no longer J1.7
- net RESET_ISO: now also U12.2; no longer U5.4
- net RQ: now also J1.5; no longer J1.6
- net SCK: now also J1.3, U5.4; no longer J1.4
- net SELECT: now also J1.9, R33.2, U6.4; no longer J1.1, U10.4
- net SETPHASE: now also U6.2; no longer U10.2
- net VDD: now also J1.7, U5.5; no longer J1.8, U$1.5
Routing:
- net GNDI: track 184.8 -> 29.9 mm, vias 9 -> 6
- net AGND: track 0.00 -> 57.4 mm, vias 0 -> 6
- net GND: track 57.8 -> 5.78 mm, vias 3 -> 4
- net VCC: track 73.8 -> 97.0 mm, vias 5 -> 3
- net LNV1: track 0.00 -> 14.3 mm
- net N$37: track 0.00 -> 13.4 mm
- net SELECT: track 0.00 -> 12.8 mm
- net SETPHASE: track 0.00 -> 11.5 mm
- net CS: track 26.3 -> 37.7 mm
- net LNV2: track 0.00 -> 10.9 mm, vias 0 -> 1
- net N$38: track 0.00 -> 8.80 mm
- net MISO_OUT: track 6.98 -> 0.00 mm
- net RESET_ISO: track 23.5 -> 30.4 mm, vias 2 -> 3
- net MISO_ISO: track 8.31 -> 15.1 mm
- net N$18: track 1.55 -> 7.94 mm
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- added copper zone on layer 1, net AGND
Other:
- board size 58 x 27 mm -> 64.5 x 35.5 mm
- board text added: "CF1"
- board text added: "CF2"
- board text added: "CalPlug, UCI"
- board text added: "SEL"
- board text added: "Watt Meter Rev.4"
- board text added: "ZX"
- board text added: "ZX_I"
- board text removed: "CalPlug"
- board text removed: "Watt Meter"
