File: Documents/Wattmeter_V4/WattMeter_v4.sch (EAGLE design)
At the start: 77 parts, among them Q1 QUARTZ_3.58M_2PIN, U1 ADE7953, U2 PAM2305, U3 ISO7241, U4 SN74LVC, U5 PS2505, U6 PS2505, U7 SN74LVC, U8 SN6501, U9 TRANSFO_3.3

Commit message: Updated V4 board
Parts:
- removed JP5: (no value), SparkFun-Connectors:M08
- removed R52: 120k, resistor:R-EU_M1206
- removed U$1: BUFFER-NL17SZ125, arducoder:BUFFER-NL17SZ125
- added J1: (no value), SparkFun-Connectors:CONN_09
- added R26, R27, R33: 4.7k, Nizanlib:0402-RES
- added R30, R31, R32: 100k, SparkFun:RESISTOR0603-RES
- added U10, U12: PS2505, wattmeter:PS2505
- added U11: SN74LVC1G3157DBVR, TI:SN74LVC1G3157DBVR
- C17, C7: value 68nF -> 0.033uF
- R12: value 120k -> 55k; device resistor:R-EU_M1206 -> SparkFun:RESISTOR0603-RES
- R14: value 10k -> 4.7K
- R18: value 499R -> 1K
- R19: value 499R -> 1k
- R25: value 220k -> 100k; device resistor:R-EU_R2010 -> SparkFun:RESISTOR0603-RES
- R28, R7: value 220k -> 4.7k; device resistor:R-EU_R2010 -> SparkFun:RESISTOR0603-RES
- R29: value 220k -> 55k; device resistor:R-EU_R2010 -> SparkFun:RESISTOR0603-RES
- U5: value PS2505 -> NL17SZ125; device Damien_divers:PS2505 -> wattmeter:NL17SZ125
- U6: device Damien_divers:PS2505 -> wattmeter:PS2505
Connections:
- removed net N$14: R12.1, R52.2
- removed net N$15: R12.2, R7.1
- removed net N$17: R25.1, R7.2
- removed net N$29: R10.1, U6.1
- removed net VN_IN: JP2.1, R29.2
- new net +3V3: U11.VCC
- new net AGND: C10.2, C11.1, C12.2, C13.1, C14.1, C17.2, C28.1, C29.2, C30.1, C31.2, C5.1, C6.2, C7.2, C8.2, R11.2, R17.1, R18.2, R19.2, R20.2, R9.1, U1.AGND
- new net CF1: U1.CF1
- new net CF2: U1.CF2
- new net LNV1: JP2.1, R30.1
- new net LNV2: JP2.2, R31.1
- new net N$13: R31.2, R32.1
- new net N$22: R29.1, R32.2
- new net N$36: R12.1, R25.2
- new net N$37: R28.1, R29.2, U11.B2
- new net N$38: R12.2, R7.2, U11.B1
- new net N$39: R10.1, U10.ANODE
- new net REVP: U1./REVP
- new net RQ: J1.5
- new net SELECT: J1.9, R26.1, R33.2, U6.COLLERTOR
- new net SETPHASE: R27.1, U11.S, U6.CATHODE
- new net ZX: U1.ZX
- new net ZX_I: U1.ZX_I
- net CS: now also J1.1, U5.!OE; no longer JP5.1, U$1.OE#
- net GND: now also J1.8, R33.1, U10.EMITTER, U12.COLLERTOR, U5.GND, U6.EMITTER; no longer JP5.8, U$1.GND, U5.2, U6.3
- net GNDI: now also R28.2, R7.1, U10.CATHODE, U11.GND, U12.ANODE, U6.ANODE; no longer C10.2, C11.1, C12.2, C13.1, C14.1, C17.2, C28.1, C29.2, C30.1, C31.2, C5.1, C6.2, C7.2, C8.2, R11.2, R17.1, R18.2, R19.2, R20.2, R9.1, U1.AGND, U5.3, U6.2
- net IRQ: now also U10.COLLERTOR; no longer JP5.5, U6.4
- net MISO: now also U5.IN; no longer U$1.IN
- net MISO_OUT: now also J1.2; no longer JP5.2, U$1.OUT
- net MOSI: now also J1.4; no longer JP5.4
- net N$25: now also U12.EMITTER; no longer U5.1
- net N$3: no longer R28.1
- net N$35: now also R25.1, R30.2; no longer R28.2, R29.1
- net RESET: now also J1.6; no longer JP5.6
- net RESET_ISO: now also U12.CATHODE; no longer U5.4
- net SCK: now also J1.3, U5.OUT; no longer JP5.3
- net V2P: no longer R52.1
- net VCC: now also R27.2
- net VDD: now also J1.7, R26.2, U5.VCC; no longer JP5.7, U$1.VCC
- net VP_IN: now also U11.A; no longer JP2.2, R25.2
Other:
- note added: "Populate Either R33 or R26 according to default direction when NC"
- moved on the sheet: C27
