File: Documents/Wattmeter_V4/WattMeter_v4.sch (EAGLE design)
At the start: 88 parts, among them Q1 QUARTZ_3.58M_2PIN, U1 ADE7953, U10 PS2505, U11 SN74LVC1G3157DBVR, U12 PS2505, U13 SN74LVC, U2 PAM2305, U3 ISO7241, U4 SN74LVC, U5 NL17SZ125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

Commit message: latest updates for I2C and SPI
Parts:
- removed R26, R33: 4.7k, Nizanlib:0402-RES
- R3: value 10k -> 4.7k
- U3: device Damien_divers:ISO7241 -> wattmeter:ISO7241
- U4: SPICEPREFIX (none) -> X
Connections:
- net IRQ renamed IRQ_OUT
- removed net +3V3: U11.VCC
- removed net N$29: U11.S, U7.OUTB
- net GND: now also R3.1, U3.GND1@3; no longer R33.1, U3.GND2
- net GNDI: now also U3.GND2, U3.GND2@3; no longer U3.ISOGND, U3.ISOGND2
- net IRQ_ISO: no longer R3.2
- net MISO: now also U3.OUTC; no longer U3.INC
- net MISO_ISO: now also U3.INC; no longer U3.OUTC
- net MISO_OUT: now also U5.OUT
- net N$40: now also R3.2
- net N$42: no longer R26.1, R33.2
- net SCK: no longer U3.INB, U5.OUT
- net SETPHASE: now also U11.S; no longer U7.INB
- net VCC: now also U11.VCC, U3.VCC2; no longer R3.1, U3.ISOVCC
- net VDD: no longer R26.2
Other:
- note added: "Analog multiplexer"
- note added: "Dual NOT gate"
- note added: "INV"
- note added: "NORM"
- note added: "Select polarity"
- note removed: "#######"
- note removed: "Populate Either R33 or R26 according to default direction when NC"
- moved on the sheet: C13, C14, C15, C16, C24, C25, R3, R34, U5
