File: Documents/Wattmeter_V4/WattMeter_v4_I2C.sch (EAGLE design)
At the start: 86 parts, among them Q1 QUARTZ_3.58M_2PIN, U1 ADE7953, U10 PS2505, U11 SN74LVC1G3157DBVR, U12 PS2505, U13 SN74LVC, U2 PAM2305, U3 ISO7241, U4 SN74LVC, U5 NL17SZ125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

Commit message: latest updates for I2C and SPI
Parts:
- removed U3: ISO7241, wattmeter:ISO7241
- removed U5: NL17SZ125, wattmeter:NL17SZ125
- added R26, R33, R35, R36: 4.7k, Nizanlib:0402-RES
- added R37, R38: 4.7K, Nizanlib:0402-RES
- added SJ1, SJ2: (no value), jumper:SJ
- added U14: ISO1541, wattmeter:ISO1541
Connections:
- removed net CS: J1.1, U3.IND, U5.!OE
- removed net MISO: U3.OUTC, U5.IN
- removed net MISO_ISO: U1.MISO, U3.INC
- removed net MISO_OUT: J1.2, U5.OUT
- removed net MOSI: J1.4, U3.INA
- removed net MOSI_ISO: U1.MOSI, U3.OUTA
- removed net SCK: J1.3
- removed net SCK_ISO: U1.SCLK, U3.OUTB
- new net N$29: R36.1, SJ1.1
- new net N$44: R35.1, SJ2.1
- new net SCL: J1.4, SJ2.2, U14.SCL1
- new net SCLK_ISO: R38.1
- new net SCL_ISO: R33.1, U1.MOSI, U1.SCLK, U14.SCL2
- new net SDA: J1.2, SJ1.2, U14.SDA1
- new net SDA_ISO: R26.1, U1.MISO, U14.SDA2
- net AGND: now also J2.3; no longer J2.1
- net CS_ISO: now also R37.1; no longer U3.OUTD
- net GND: now also U14.GND1; no longer U3.GND1, U3.GND1@3, U5.GND
- net GNDI: now also U14.GND2; no longer U3.GND2, U3.GND2@3
- net LNV1: now also J2.1; no longer J2.2
- net LNV2: now also J2.2; no longer J2.3
- net VCC: now also R26.2, R33.2, R37.2, R38.2, U14.VCC2; no longer U3.EN2, U3.VCC2
- net VDD: now also R35.2, R36.2, U14.VCC1; no longer U3.EN1, U3.VCC1, U5.VCC
Other:
- note added: "Analog multiplexer"
- note added: "I2C resistor enable"
- note added: "INV"
- note added: "NORM"
- note added: "Select polarity"
- note removed: "ISO7241"
- note removed: "SCL"
- note removed: "SDA"
- moved on the sheet: C24, C25, R14, U10, U12, U6
